Commit message: Gripper joints mimicing one direction

File: kassow_robot_dev/pkg_kassowa_robot/urdf/kr1410.urdf (robot description, URDF)
Before this commit: robot kr1410, 10 links, 9 joints
Links:
- added link ee_link
Joints:
- added joint ee_joint: type fixed, parent tool_io, child ee_link, origin xyz=0 0 0.05 rpy=0 0 0
- joint joint_tool_io: origin xyz=0 0.053 -0.0465 rpy=1.5708 -1.5708 0 -> xyz=0 0.053 -0.0465 rpy=1.5708 -1.5708 3.14

File: kassow_robot_dev/pkg_kassowa_robot/urdf/kr1410_gazebo.xacro (robot description, xacro)
@@ -16,10 +16,10 @@
     <xacro:self_collision link="link_6"/>
     <xacro:self_collision link="tool_io"/>
-        <gazebo>
-            <plugin name="ros_control" filename="libgazebo_ros_control.so">
-                <!--robotNamespace>/</robotNamespace-->
-                <!--robotSimType>gazebo_ros_control/DefaultRobotHWSim</robotSimType-->
-            </plugin>
-        </gazebo>
+    <gazebo>
+        <plugin name="ros_control" filename="libgazebo_ros_control.so">
+            <!--robotNamespace>/</robotNamespace-->
+            <!--robotSimType>gazebo_ros_control/DefaultRobotHWSim</robotSimType-->
+        </plugin>
+    </gazebo>
     <!-- Define the kr1410 robot position and orientation in the world coordinate system -->
     <link name="world"/>

File: kassow_robot_dev/pkg_kassowa_robot/urdf/kr1410_macro.xacro (robot description, xacro)
@@ -12,3 +12,10 @@
         <origin rpy="0 0 0" xyz="0 0 0"/>
     </joint>
+    <!-- Create end effector link -->
+    <link name="ee_link"/>
+    <joint name="ee_joint" type="fixed">
+        <parent link="tool_io"/>
+        <child link="ee_link"/>
+        <origin rpy="0 0 0" xyz="0 0 0.05"/>
+    </joint>
 </robot>

File: kassow_robot_dev/pkg_kassowa_robot/urdf/kr1410_model.xacro (robot description, xacro)
@@ -233,5 +233,5 @@
   </link>
   <joint name="joint_tool_io" type="revolute">
-    <origin rpy="1.5708 -1.5708 0" xyz="0 0.053 -0.0465"/>
+    <origin rpy="1.5708 -1.5708 3.14" xyz="0 0.053 -0.0465"/>
     <parent link="link_6"/>
     <child link="tool_io"/>

File: kassow_robot_dev/robotiq_2f_85_gripper_visualization/urdf/robotiq_arg2f_85_model_macro.xacro (robot description, xacro)
@@ -4,9 +4,9 @@
   <xacro:macro name="outer_knuckle" params="prefix fingerprefix stroke">
     <link name="${prefix}${fingerprefix}_outer_knuckle">
-      <!--<inertial>
+      <inertial>
         <origin xyz="-0.000200000000003065 0.0199435877845359 0.0292245259211331" rpy="0 0 0" />
         <mass value="0.00853198276973456" />
         <inertia ixx="2.89328108496468E-06" ixy="-1.57935047237397E-19" ixz="-1.93980378593255E-19" iyy="1.86719750325683E-06" iyz="-1.21858577871576E-06" izz="1.21905238907251E-06" />
-        </inertial> -->
+      </inertial>
       <visual>
         <origin xyz="0 0 0" rpy="0 0 0" />
@@ -28,9 +28,9 @@
   <xacro:macro name="outer_finger" params="prefix fingerprefix stroke">
     <link name="${prefix}${fingerprefix}_outer_finger">
-      <!--<inertial>
+      <inertial>
         <origin xyz="0.00030115855001899 0.0373907951953854 -0.0208027427000385" rpy="0 0 0" />
         <mass value="0.022614240507152" />
         <inertia ixx="1.52518312458174E-05" ixy="9.76583423954399E-10" ixz="-5.43838577022588E-10" iyy="6.17694243867776E-06" iyz="6.78636130740228E-06" izz="1.16494917907219E-05" />
-        </inertial> -->
+      </inertial>
       <visual>
         <origin xyz="0 0 0" rpy="0 0 0" />
@@ -52,9 +52,9 @@
   <xacro:macro name="inner_knuckle" params="prefix fingerprefix stroke">
     <link name="${prefix}${fingerprefix}_inner_knuckle">
-      <!--<inertial>
+      <inertial>
         <origin xyz="0.000123011831763771 0.0507850843201817 0.00103968640075166" rpy="0 0 0" />
        <mass value="0.0271177346495152" />
         <inertia ixx="2.61910379223783E-05" ixy="-2.43616858946494E-07" ixz="-6.37789906117123E-09" iyy="2.8270243746167E-06" iyz="-5.37200748039765E-07" izz="2.83695868220296E-05" />
-        </inertial> -->
+      </inertial>
       <visual>
         <origin xyz="0 0 0" rpy="0 0 0" />
@@ -76,9 +76,9 @@
   <xacro:macro name="inner_finger" params="prefix fingerprefix stroke">
     <link name="${prefix}${fingerprefix}_inner_finger">
-      <!--<inertial>
+      <inertial>
         <origin xyz="0.000299999999999317 0.0160078233491243 -0.0136945669206257" rpy="0 0 0" />
         <mass value="0.0104003125914103" />
         <inertia ixx="2.71909453810972E-06" ixy="1.35402465472579E-21" ixz="-7.1817349065269E-22" iyy="7.69100314106116E-07" iyz="6.74715432769696E-07" izz="2.30315190420171E-06" />
-        </inertial> -->
+      </inertial>
       <visual>
         <origin xyz="0 0 0" rpy="0 0 0" />
@@ -101,4 +101,9 @@
   <xacro:macro name="inner_finger_pad" params="prefix fingerprefix">
     <link name="${prefix}${fingerprefix}_inner_finger_pad">
+      <inertial>
+        <origin xyz="0.0000299999999999317 0.00160078233491243 -0.00136945669206257" rpy="0 0 0" />
+        <mass value="0.00104003125914103" />
+        <inertia ixx="2.71909453810972E-07" ixy="1.35402465472579E-22" ixz="-7.1817349065269E-23" iyy="7.69100314106116E-08" iyz="6.74715432769696E-08" izz="2.30315190420171E-07" />
+      </inertial>
       <visual>
         <origin xyz="0 0 0" rpy="0 0 0" />
