Commit message: create mir_ur5e_ar autonomous robot package

File: kassow_robot_dev/pkg_kr_sim/urdf/gazebo.xacro (robot description, xacro)
@@ -13,4 +13,5 @@
         </gazebo>
     </xacro:macro>
+    <!-- Self collision in gazebo for robotic arm -->
     <xacro:self_collision link="base_link_1"/>
     <xacro:self_collision link="link_1"/>
@@ -21,22 +22,4 @@
     <xacro:self_collision link="link_6"/>
     <xacro:self_collision link="tool_io"/>
-    <!-- Define the kr1410 robot position and orientation in the world coordinate system -->
-    <link name="world"/>
-    <joint name="world_joint" type="fixed">
-        <parent link="world"/>
-        <child link="base_link"/>
-        <origin rpy="0.0 0.0 0.0" xyz="0.0 0.0 1.0"/>
-    </joint>
-    <!-- <xacro:self_collision link="robotiq_arg2f_base_link"/>
-    <xacro:self_collision link="left_outer_knuckle"/>
-    <xacro:self_collision link="left_outer_finger"/>
-    <xacro:self_collision link="left_inner_finger"/>
-    <xacro:self_collision link="left_inner_finger_pad"/>
-    <xacro:self_collision link="left_inner_knuckle"/>
-    <xacro:self_collision link="right_outer_knuckle"/>
-    <xacro:self_collision link="right_outer_finger"/>
-    <xacro:self_collision link="right_inner_finger"/>
-    <xacro:self_collision link="right_inner_finger_pad"/>
-    <xacro:self_collision link="right_inner_knuckle"/> -->
     <!-- Gazebo Plugins -->
     <gazebo>
@@ -48,5 +31,5 @@
     <!-- loading plugin: mimic joints works in gazebo now-->
     <xacro:property name="parent_joint" value="finger_joint"/>
-    <xacro:macro name="mimic_joint_plugin_gazebo" params="parent_joint:=${parent_joint} mimic_joint has_pid:=true multiplier:=1.0 offset:=0.0 max_effort:=5.0 sensitiveness:=0.0 robot_namespace:=''">
+    <xacro:macro name="mimic_joint_plugin_gazebo" params="parent_joint:=${parent_joint} mimic_joint has_pid:=false multiplier:=1.0 offset:=0.0 max_effort:=5.0 sensitiveness:=0.0 robot_namespace:=''">
         <gazebo>
             <plugin name="${mimic_joint}_mimic_plugin" filename="libroboticsgroup_upatras_gazebo_mimic_joint_plugin.so">
@@ -72,17 +55,33 @@
     <xacro:mimic_joint_plugin_gazebo mimic_joint="right_inner_knuckle_joint" multiplier="1.0"/>
     <gazebo>
-        <disable_collisions link1="right_outer_finger" link2="robotiq_arg2f_base_link" reason="Adjacent"/>
-        <disable_collisions link1="right_outer_knuckle" link2="right_inner_knuckle" reason="Adjacent"/>
-        <disable_collisions link1="right_outer_knuckle" link2="right_outer_finger" reason="Adjacent"/>
-        <disable_collisions link1="right_outer_finger" link2="right_inner_finger" reason="Adjacent"/>
-        <disable_collisions link1="right_inner_knuckle" link2="right_inner_finger" reason="Adjacent"/>
-        <disable_collisions link1="left_outer_knuckle" link2="robotiq_arg2f_base_link" reason="Adjacent"/>
-        <disable_collisions link1="left_inner_knuckle" link2="robotiq_arg2f_base_link" reason="Adjacent"/>
-        <disable_collisions link1="left_outer_knuckle" link2="robotiq_arg2f_base_link" reason="Adjacent"/>
-        <disable_collisions link1="left_outer_finger" link2="robotiq_arg2f_base_link" reason="Adjacent"/>
-        <disable_collisions link1="left_outer_knuckle" link2="left_inner_knuckle" reason="Adjacent"/>
-        <disable_collisions link1="left_outer_knuckle" link2="left_outer_finger" reason="Adjacent"/>
-        <disable_collisions link1="left_outer_finger" link2="left_inner_finger" reason="Adjacent"/>
-        <disable_collisions link1="left_inner_knuckle" link2="left_inner_finger" reason="Adjacent"/>
+        <plugin name="gazebo_grasp_fix" filename="libgazebo_grasp_fix.so">
+            <arm>
+                <arm_name>kr1410_robot</arm_name>
+                <palm_link>left_outer_knuckle</palm_link>
+                <palm_link>right_outer_knuckle</palm_link>
+                <gripper_link>left_inner_finger</gripper_link>
+                <gripper_link>right_inner_finger</gripper_link>
+            </arm>
+        <forces_angle_tolerance>100</forces_angle_tolerance>
+        <update_rate>4</update_rate>
+        <grip_count_threshold>4</grip_count_threshold>
+        <max_grip_count>8</max_grip_count>
+        <release_tolerance>0.005</release_tolerance>
+        <disable_collisions_on_attach>false</disable_collisions_on_attach>
+        <contact_topic>__default_topic__</contact_topic>
+        </plugin>
     </gazebo>
+    <!-- Define the kr1410 robot position and orientation in the world coordinate system -->
+    <link name="world"/>
+    <joint name="world_joint" type="fixed">
+        <parent link="world"/>
+        <child link="base_link"/>
+        <origin rpy="0.0 0.0 0.0" xyz="0.0 0.0 1.0"/>
+    </joint>
+    <joint name="pedestal_joint" type="fixed">
+        <!-- <origin rpy="0 0 0" xyz="0.5 1.8 0.0"/> -->
+        <origin rpy="0 0 0" xyz="0.0 0.0 0.0"/>
+        <parent link="world"/>
+        <child link="pedestal_link"/>
+    </joint>
 </robot>

File: kassow_robot_dev/pkg_kr_sim/urdf/kr1410_gripper.xacro (robot description, xacro)
@@ -2,7 +2,8 @@
 <robot name="kr1410_robot" xmlns:xacro="http://wiki.ros.org/xacro">
     <!-- Author: Shivam -->
-    <xacro:include filename="$(find pkg_kassowa_robot)/urdf/kr1410_model.xacro"/>
-    <xacro:include filename="$(find pkg_kassowa_robot)/urdf/kr1410_transmissions.xacro"/>
-    <xacro:include filename="$(find robotiq_2f_85_gripper_visualization)/urdf/robotiq_arg2f_85_model.xacro"/>
+    <xacro:include filename="$(find kr1410_cobot)/urdf/kr1410_model.xacro"/>
+    <xacro:include filename="$(find kr1410_cobot)/urdf/kr1410_transmissions.xacro"/>
+    <xacro:include filename="$(find robotiq_2f_85_gripper)/urdf/robotiq_arg2f_85_model_macro.xacro" />
+    <xacro:robotiq_arg2f_85 parent="ee_link" prefix=""/>
     <xacro:include filename="$(find pkg_kr_sim)/urdf/gazebo.xacro"/>
     <!-- Create a dummy link base_link -->
@@ -35,22 +36,10 @@
         </inertial>
     </link>
-    <joint name="pedestal_joint" type="fixed">
-        <!-- <origin rpy="0 0 0" xyz="0.5 1.8 0.0"/> -->
-        <origin rpy="0 0 0" xyz="0.0 0.0 0.0"/>
-        <parent link="world"/>
-        <child link="pedestal_link"/>
-    </joint>
-    <!-- Create end effector link -->
+    <!-- Create end effector link. On this link gripper will be mounted -->
     <link name="ee_link"/>
     <joint name="ee_joint" type="fixed">
         <parent link="tool_io"/>
         <child link="ee_link"/>
-        <origin rpy="0 0 0" xyz="0 0 0.05"/>
-    </joint>
-    <!-- Attach Robotiq Gripper to Kassow Robot -->
-    <joint name="gripper_joint" type="fixed">
-        <parent link="ee_link"/>
-        <child link="robotiq_arg2f_base_link"/>
-        <origin rpy="0 0 0" xyz="0 0 0"/>
+        <origin rpy="0 0 0" xyz="0 0 0.0465"/>
     </joint>
 </robot>

File: kassow_robot_dev/robot_description/robotiq_2f_85_gripper/urdf/robotiq_arg2f.urdf (robot description, URDF)
Before this commit: robot kr1410_robot, 24 links, 23 joints
Links:
- removed link base_link_1
- removed link ee_link
- removed link link_1
- removed link link_2
- removed link link_3
- removed link link_4
- removed link link_5
- removed link link_6
- removed link pedestal_link
- removed link tool_io
Joints:
- removed joint base_link_joint
- removed joint ee_joint
- removed joint joint_1
- removed joint joint_2
- removed joint joint_3
- removed joint joint_4
- removed joint joint_5
- removed joint joint_6
- removed joint joint_tool_io
- removed joint pedestal_joint
- joint gripper_base_joint: parent ee_link -> base_link
- joint tool_frame_joint: parent ee_link -> base_link
- joint world_joint: origin xyz=0.0 0.0 1.0 rpy=0.0 0.0 0.0 -> xyz=0.0 0.0 0.1 rpy=0.0 0.0 0.0
