Commit message: MIR UR5 started

File: pkg_ur5e_r/urdf/mounted_ur5e.urdf (robot description, URDF)
Before this commit: robot mounted_ur5e, 15 links, 14 joints
Links:
- link schunk_gripper: geometry collision mesh filename=package://schunk_gripper/meshes/visual/schunk_gripper.dae; visual mesh filename=package://schunk_gripper/meshes/visual/schunk_gripper.dae

File: pkg_ur5e_r/urdf/mounted_ur5e.xacro (robot description, xacro)
@@ -6,5 +6,5 @@
     <xacro:include filename="$(find ur_description)/urdf/ur5e.xacro"/>
     <!-- End effector -->
-    <xacro:include filename="$(find pkg_ur5e_r)/urdf/schunk_gripper.xacro"/>
+    <xacro:include filename="$(find schunk_gripper)/urdf/schunk_gripper.xacro"/>
     <!-- Gazebo settings -->
     <xacro:include filename="$(find pkg_ur5e_r)/urdf/ur5e_gazebo.xacro"/>
